File: M.I.A. PCB/M.I.A..kicad_pcb (KiCad board)
At the start: 4 copper layers, 50.8 x 106.6 mm, 178 parts, among them J1 USB_C_Receptacle_USB2.0_16P, J10 Conn_01x03, J11 Conn_01x03, J12 MSD-4-A, J13 Conn_01x04_Socket, J14 Conn_01x03, J15 Conn_01x03, J16 Conn_01x03, J17 Conn_01x03, J18 Conn_01x04_Socket, J19 Conn_01x04_Socket, J2 Conn_Coaxial, J20 Screw_Terminal_01x02, J21 Screw_Terminal_01x02, J22 Screw_Terminal_01x02, J23 Screw_Terminal_01x02, J24 Conn_01x04_Socket, J25 Conn_01x08_Socket, J26 Conn_01x04_Socket, J27 Conn_01x02_Socket, J28 Conn_01x04_Socket, J29 Conn_01x02_Socket, J3 Screw_Terminal_01x02, J30 Conn_01x02_Socket, J31 Conn_01x02_Socket, J32 Screw_Terminal_01x02, J33 Screw_Terminal_01x02, J4 Screw_Terminal_01x02, J5 Conn_01x02_Pin, J6 Conn_01x04_Socket, J7 Conn_01x03, J8 Conn_01x03, J9 Conn_01x04_Socket, Q1 AO3400A, Q2 AO3400A, Q3 AO3400A, Q4 AO3400A, SW1 SW_Push, SW2 SW_Push, U1 W25Q128JVS, U10 INA219AxDCN, U11 AP2112K-3.3, U12 AP62150WU, U13 TPS2121RUXR, U14 AP62150WU, U15 74AHC541, U2 RP2350B-QFN80, U3 MMC5983MA, U4 ICM-45686, U5 MS5611-01BA, U6 TMP117xxDRV, U7 MAX-M10S, U8 KX134-1211, U9 TPS2121RUXR, Y1 ABM8-272-T3

Commit message: Likely Final PCB
Parts:
- added C44: 100u, Capacitor_THT:C_Radial_D5.0mm_H11.0mm_P2.00mm, F.Cu at (66.8, 112.0)
- added C45: 100u, Capacitor_THT:C_Radial_D5.0mm_H11.0mm_P2.00mm, F.Cu at (24.0, 112.0)
- added C46: 100n, Capacitor_SMD:C_0603_1608Metric, B.Cu at (64.2, 115.8)
- added C47: 100n, Capacitor_SMD:C_0603_1608Metric, B.Cu at (53.0, 115.8)
- added C48: 100n, Capacitor_SMD:C_0603_1608Metric, B.Cu at (37.9, 115.8)
- added C49: 100n, Capacitor_SMD:C_0603_1608Metric, B.Cu at (26.6, 115.8)
- renumbered REF** to G1, REF** to G2, REF** to G3
Routing:
- net VSYS: track 4.17 -> 53.4 mm, vias 13 -> 16
- net +3.3V: track 176.7 -> 186.5 mm
- net SPI_MISO_TLM: track 85.6 -> 79.5 mm
- net /D+: track 16.6 -> 11.0 mm
- net SPI_MOSI_TLM: track 76.9 -> 81.4 mm
- net SPI_SCK_TLM: track 96.5 -> 98.5 mm
- net SPI_CS_TLM: track 79.2 -> 77.9 mm
- net /Peripherals/servo6: track 33.6 -> 34.7 mm
- net /Peripherals/servo4: track 34.6 -> 35.5 mm
- net GND: vias 146 -> 144
- added copper zone on In2.Cu, net +3.3V
Other:
- board text added: "M.I.A. V1.0 6/26 Landon Doughty"
