File: M.I.A. PCB/M.I.A..kicad_pcb (KiCad board)
At the start: 4 copper layers, 50.8 x 106.6 mm, 184 parts, among them J1 USB_C_Receptacle_USB2.0_16P, J10 Conn_01x03, J11 Conn_01x03, J12 MSD-4-A, J13 Conn_01x04_Socket, J14 Conn_01x03, J15 Conn_01x03, J16 Conn_01x03, J17 Conn_01x03, J18 Conn_01x04_Socket, J19 Conn_01x04_Socket, J2 Conn_Coaxial, J20 Screw_Terminal_01x02, J21 Screw_Terminal_01x02, J22 Screw_Terminal_01x02, J23 Screw_Terminal_01x02, J24 Conn_01x04_Socket, J25 Conn_01x08_Socket, J26 Conn_01x04_Socket, J27 Conn_01x02_Socket, J28 Conn_01x04_Socket, J29 Conn_01x02_Socket, J3 Screw_Terminal_01x02, J30 Conn_01x02_Socket, J31 Conn_01x02_Socket, J32 Screw_Terminal_01x02, J33 Screw_Terminal_01x02, J4 Screw_Terminal_01x02, J5 Conn_01x02_Pin, J6 Conn_01x04_Socket, J7 Conn_01x03, J8 Conn_01x03, J9 Conn_01x04_Socket, Q1 AO3400A, Q2 AO3400A, Q3 AO3400A, Q4 AO3400A, SW1 SW_Push, SW2 SW_Push, U1 W25Q128JVS, U10 INA219AxDCN, U11 AP2112K-3.3, U12 AP62150WU, U13 TPS2121RUXR, U14 AP62150WU, U15 74AHC541, U2 RP2350B-QFN80, U3 MMC5983MA, U4 ICM-45686, U5 MS5611-01BA, U6 TMP117xxDRV, U7 MAX-M10S, U8 KX134-1211, U9 TPS2121RUXR, Y1 ABM8-272-T3

Commit message: Routing Updates
Parts:
- R2, R3: value 27 -> 33
- R25, R6: value 270 -> 330
Other:
- board text added: "D0"
Changed lines of the file:
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@@
 			)
 		)
-		(property "Value" "270"
+		(property "Value" "330"
 			(at 0 1.43 0)
 			(layer "F.Fab")
@@
 			)
 		)
-		(property "Value" "27"
+		(property "Value" "33"
 			(at 0 1.43 0)
 			(layer "F.Fab")
@@
 			)
 		)
-		(property "Value" "27"
+		(property "Value" "33"
 			(at 0 1.43 0)
 			(layer "F.Fab")
@@
 			)
 		)
-		(property "Value" "270"
+		(property "Value" "330"
 			(at 0 -1.43 0)
 			(layer "B.Fab")
@@
 		(layer "Edge.Cuts")
 	)
+	(gr_text "MISO"
+		(at 26 71.35 0)
+		(layer "F.SilkS")
+		(effects
+			(font
+				(size 0.8 0.8)
+				(thickness 0.15)
+			)
+			(justify left)
+		)
+	)
 	(gr_text "+"
 		(at 27.5 85.5 0)
@@
 		)
 	)
+	(gr_text "D0"
+		(at 26 69.3 0)
+		(layer "F.SilkS")
+		(effects
+			(font
+				(size 0.8 0.8)
+				(thickness 0.15)
+			)
+			(justify left)
+		)
+	)
 	(gr_text "2"
 		(at 65.7 36 0)
@@
 		)
 	)
+	(gr_text "RST"
+		(at 26 74.35 0)
+		(layer "F.SilkS")
+		(effects
+			(font
+				(size 0.8 0.8)
+				(thickness 0.15)
+			)
+			(justify left)
+		)
+	)
 	(gr_text "+"
 		(at 27.5 106.55 0)
@@
 		)
 	)
+	(gr_text "+"
+		(at 66.75 114 90)
+		(layer "F.SilkS")
+		(effects
+			(font
+				(size 0.8 0.8)
+				(thickness 0.15)
+			)
+			(justify left)
+		)
+	)
 	(gr_text "SDA"
 		(at 25.1 58.6 0)
@@
 		)
 	)
+	(gr_text "SCK"
+		(at 26 70.3 0)
+		(layer "F.SilkS")
+		(effects
+			(font
+				(size 0.8 0.8)
+				(thickness 0.15)
+			)
+			(justify left)
+		)
+	)
 	(gr_text "5V"
 		(at 28.6 83.75 0)
@@
 		)
 	)
+	(gr_text "-"
+		(at 68.7 114 90)
+		(layer "F.SilkS")
+		(effects
+			(font
+				(size 0.8 0.8)
+				(thickness 0.15)
+			)
+			(justify left)
+		)
+	)
 	(gr_text "SPI0"
 		(at 28.5 37.4 0)
@@
 		)
 	)
+	(gr_text "-"
+		(at 26 68.3 0)
+		(layer "F.SilkS")
+		(effects
+			(font
+				(size 0.8 0.8)
+				(thickness 0.15)
+			)
+			(justify left)
+		)
+	)
 	(gr_text "27"
 		(at 47.55 20 270)
@@
 	)
 	(gr_text "+"
+		(at 24.05 112.85 270)
+		(layer "F.SilkS")
+		(effects
+			(font
+				(size 0.8 0.8)
+				(thickness 0.15)
+			)
+			(justify left)
+		)
+	)
+	(gr_text "+"
 		(at 65.7 27.7 0)
 		(layer "F.SilkS")
@@
 		)
 	)
+	(gr_text "MOSI"
+		(at 26 72.3 0)
+		(layer "F.SilkS")
+		(effects
+			(font
+				(size 0.8 0.8)
+				(thickness 0.15)
+			)
+			(justify left)
+		)
+	)
+	(gr_text "-"
+		(at 22.1 112.85 270)
+		(layer "F.SilkS")
+		(effects
+			(font
+				(size 0.8 0.8)
+				(thickness 0.15)
+			)
+			(justify left)
+		)
+	)
 	(gr_text "8|7|6|5"
 		(at 32.275 109.55 0)
@@
 		)
 	)
+	(gr_text "+"
+		(at 26 67.3 0)
+		(layer "F.SilkS")
+		(effects
+			(font
+				(size 0.8 0.8)
+				(thickness 0.15)
+			)
+			(justify left)
+		)
+	)
+	(gr_text "CS"
+		(at 26 73.3 0)
+		(layer "F.SilkS")
+		(effects
+			(font
+				(size 0.8 0.8)
+				(thickness 0.15)
+			)
+			(justify left)
+		)
+	)

Commit message: Added Test Points + Back Graphics
Parts:
- added C50: 10u, Capacitor_SMD:C_0805_2012Metric, B.Cu at (36.7, 87.1)
- added C51: 100n, Capacitor_SMD:C_0603_1608Metric, F.Cu at (50.1, 87.8)
- D6, D7, D8, D9: value BZT52Bxx -> BZT52C6V2
- R18, R27: value 47K -> 47k
- R19: value 2m -> 5m
- R38, R39, R46, R47: value 5M -> 50k
- R43, R45, R51, R53: value 1M -> 10k
- R7, R8: value 4.7k -> 5.1k
- U15: value 74AHC541 -> 74AHCT541
Connections:
- U2 pad 11: UART0_TX -> SPI_MISO_SEN
- U2 pad 12: UART0_RX -> LEDs
- U2 pad 13: LEDs -> SPI_SCK_SEN
- U2 pad 14: IMU_INT1 -> SPI_MOSI_SEN
- U2 pad 16: SPI_MISO_SEN -> IMU_INT1
- U2 pad 18: SPI_SCK_SEN -> UART0_TX
- U2 pad 19: SPI_MOSI_SEN -> UART0_RX
Routing:
- net IMU_INT1: track 20.6 -> 16.5 mm, vias 2 -> 0
- net Net-(U14-FB): track 0.00 -> 3.90 mm
- net Net-(U12-FB): track 0.00 -> 3.90 mm
- net SPI_MISO_SEN: track 62.5 -> 66.3 mm, vias 4 -> 5
- net SPI_SCK_SEN: track 66.8 -> 70.2 mm
- net GND: track 145.3 -> 148.0 mm
- net SPI_MOSI_SEN: track 74.9 -> 77.3 mm, vias 1 -> 3
- net +5V: track 69.3 -> 71.6 mm
- net SDA: track 106.3 -> 107.7 mm
- net SCL: track 99.9 -> 100.6 mm
- removed copper zone on B.Cu, net Net-(U12-FB)
- removed copper zone on B.Cu, net Net-(U14-FB)
