File: M.I.A. PCB/peripherals.kicad_sch (KiCad schematic)
At the start: 69 parts, among them J10 Conn_01x03, J11 Conn_01x03, J12 Screw_Terminal_01x02, J13 Screw_Terminal_01x02, J15 Screw_Terminal_01x02, J16 Screw_Terminal_01x02, J17 Screw_Terminal_01x02, J19 Conn_01x08_Socket, J20 Screw_Terminal_01x02, J21 Conn_01x04_Socket, J22 Conn_01x04_Socket, J23 Conn_01x04_Socket, J24 Conn_01x04_Socket, J25 Conn_01x04_Socket, J26 Conn_01x02_Socket, J27 Conn_01x02_Socket, J28 Conn_01x02_Socket, J29 Conn_01x02_Socket, J3 Conn_01x03, J30 Conn_01x04_Socket, J31 Conn_01x04_Socket, J32 Conn_01x04_Socket, J4 Conn_01x03, J5 Conn_01x03, J6 Conn_01x03, J7 MSD-4-A, J8 Conn_01x03, J9 Conn_01x03, Q1 AO3400A, Q2 AO3400A, Q3 AO3400A, Q4 AO3400A, U15 74AHC541

Commit message: Updated top connectors to be TLM_SPI
Parts:
- renumbered C38 to C41, C39 to C42, C40 to C43, D4 to D6, D5 to D7, D3 to D8, D6 to D9, F3 to F2, F2 to F3, J5 to J10, J6 to J11, J7 to J12, J22 to J13, J8 to J14, J9 to J15, J10 to J16, J11 to J17, J23 to J18, J25 to J19, J12 to J20, J20 to J21, J13 to J22, J16 to J23, J32 to J24, J19 to J25, J30 to J26, J29 to J27, J31 to J28, J28 to J29, J27 to J30, J26 to J31, J15 to J32, J17 to J33, J24 to J6, J3 to J7, J4 to J8, J21 to J9, JP2 to JP1, Q3 to Q2, Q2 to Q3, R28 to R32, R29 to R33, R30 to R34, R31 to R35, R32 to R36, R33 to R37, R36 to R38, R42 to R39, R34 to R40, R43 to R41, R35 to R42, R37 to R43, R38 to R46, R46 to R47, R39 to R48, R47 to R49, R40 to R50, R41 to R51, R48 to R52, R49 to R53
Connections:
- net ACC_INT is gone; now on net RST_TLM: J28.1 (Pin_1)
- net IMU_INT1 is gone; now on net +3.3V: J24.4 (Pin_4)
- net MAG_INT is gone; now on net SPI_CS_TLM: J28.2 (Pin_2)
- net +3.3V: no longer J24.2 (Pin_2), J28.3 (Pin_3)
- net D0_TLM: now also J24.2 (Pin_2)
- net GND: now also J24.3 (Pin_3); no longer J24.1 (Pin_1), J28.4 (Pin_4)
- net LEDs: no longer J24.3 (Pin_3)
- net SPI_MISO_TLM: now also J28.4 (Pin_4)
- net SPI_MOSI_TLM: now also J28.3 (Pin_3)
- net SPI_SCK_TLM: now also J24.1 (Pin_1)
Other:
- moved on the sheet: J24, J28

Commit message: Final Fixes, impedances, silkscreen etc
Connections:
- net RST_TLM: now also J24.1 (Pin_1); no longer J28.1 (Pin_1)
- net SPI_MISO_TLM: now also J28.1 (Pin_1); no longer J28.4 (Pin_4)
- net SPI_MOSI_TLM: now also J28.4 (Pin_4); no longer J28.3 (Pin_3)
- net SPI_SCK_TLM: now also J28.3 (Pin_3); no longer J24.1 (Pin_1)
Changed lines of the file:
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@@
 	(global_label "SPI_SCK_TLM"
 		(shape input)
-		(at 313.69 130.81 180)
-		(fields_autoplaced yes)
-		(effects
-			(font
-				(size 1.27 1.27)
-			)
-			(justify right)
-		)
-		(property "Intersheetrefs" "${INTERSHEET_REFS}"
-			(at 298.4887 130.81 0)
+		(at 313.69 135.89 180)
+		(fields_autoplaced yes)
+		(effects
+			(font
+				(size 1.27 1.27)
+			)
+			(justify right)
+		)
+		(property "Intersheetrefs" "${INTERSHEET_REFS}"
+			(at 299.7587 135.89 0)
 			(effects
 				(font
@@
 	(global_label "SPI_MISO_TLM"
 		(shape output)
-		(at 313.69 133.35 180)
-		(fields_autoplaced yes)
-		(effects
-			(font
-				(size 1.27 1.27)
-			)
-			(justify right)
-		)
-		(property "Intersheetrefs" "${INTERSHEET_REFS}"
-			(at 297.642 133.35 0)
+		(at 313.69 140.97 180)
+		(fields_autoplaced yes)
+		(effects
+			(font
+				(size 1.27 1.27)
+			)
+			(justify right)
+		)
+		(property "Intersheetrefs" "${INTERSHEET_REFS}"
+			(at 297.642 140.97 0)
 			(effects
 				(font
@@
 	(global_label "SPI_MOSI_TLM"
 		(shape input)
-		(at 313.69 135.89 180)
-		(fields_autoplaced yes)
-		(effects
-			(font
-				(size 1.27 1.27)
-			)
-			(justify right)
-		)
-		(property "Intersheetrefs" "${INTERSHEET_REFS}"
-			(at 297.642 135.89 0)
+		(at 313.69 133.35 180)
+		(fields_autoplaced yes)
+		(effects
+			(font
+				(size 1.27 1.27)
+			)
+			(justify right)
+		)
+		(property "Intersheetrefs" "${INTERSHEET_REFS}"
+			(at 302.843 133.35 0)
 			(effects
 				(font
@@
 	(global_label "RST_TLM"
 		(shape input)
-		(at 313.69 140.97 180)
-		(fields_autoplaced yes)
-		(effects
-			(font
-				(size 1.27 1.27)
-			)
-			(justify right)
-		)
-		(property "Intersheetrefs" "${INTERSHEET_REFS}"
-			(at 302.843 140.97 0)
+		(at 313.69 130.81 180)
+		(fields_autoplaced yes)
+		(effects
+			(font
+				(size 1.27 1.27)
+			)
+			(justify right)
+		)
+		(property "Intersheetrefs" "${INTERSHEET_REFS}"
+			(at 298.4887 130.81 0)
 			(effects
 				(font
@@
 		)
 		(property "Intersheetrefs" "${INTERSHEET_REFS}"
-			(at 299.7587 138.43 0)
-			(effects
-				(font
+			(at 297.642 138.43 0)
+			(effects
+				(font

Commit message: More Small Updates/Improvements
Other:
- note added: "I2C Connectors"
- note added: "Ignition Lines"
- note added: "MISC Conns"
- note added: "Other Connectors"
- note added: "PWR connectors"
- note added: "RGB LEDs"
- note added: "SWD Connectors"
- note added: "Secondary Radio connector"
- note added: "Sensor SPI Conn"
- note added: "UART Connector"
- note removed: "High Current Switching"
- moved on the sheet: C41, C42, C43, D10, D11, J10, J11, J12, J13, J14, J15, J16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

Commit message: Likely Final PCB
Parts:
- added C44, C45: 100u, Capacitor_THT:C_Radial_D5.0mm_H11.0mm_P2.00mm, symbol Device:C
- added C46, C47, C48, C49: 100n, Capacitor_SMD:C_0603_1608Metric, symbol Device:C
Connections:
- net GND: now also C44.2, C45.2, C46.2, C47.2, C48.2, C49.2
- net VSYS: now also C44.1, C45.1, C46.1, C47.1, C48.1, C49.1
Other:
- moved on the sheet: J10, J14, J16, J7, U15
