File: M.I.A. PCB/peripherals.kicad_sch (KiCad schematic)
At the start: 75 parts, among them J10 Conn_01x03, J11 Conn_01x03, J12 MSD-4-A, J13 Conn_01x04_Socket, J14 Conn_01x03, J15 Conn_01x03, J16 Conn_01x03, J17 Conn_01x03, J18 Conn_01x04_Socket, J19 Conn_01x04_Socket, J20 Screw_Terminal_01x02, J21 Screw_Terminal_01x02, J22 Screw_Terminal_01x02, J23 Screw_Terminal_01x02, J24 Conn_01x04_Socket, J25 Conn_01x08_Socket, J26 Conn_01x04_Socket, J27 Conn_01x02_Socket, J28 Conn_01x04_Socket, J29 Conn_01x02_Socket, J30 Conn_01x02_Socket, J31 Conn_01x02_Socket, J32 Screw_Terminal_01x02, J33 Screw_Terminal_01x02, J6 Conn_01x04_Socket, J7 Conn_01x03, J8 Conn_01x03, J9 Conn_01x04_Socket, Q1 AO3400A, Q2 AO3400A, Q3 AO3400A, Q4 AO3400A, U15 74AHC541

Commit message: Added Test Points + Back Graphics
Parts:
- added C51: 100n, Capacitor_SMD:C_0603_1608Metric, symbol Device:C
- D6, D7, D8, D9: value BZT52Bxx -> BZT52C6V2
- R38, R39, R46, R47: value 5M -> 50k
- R43, R45, R51, R53: value 1M -> 10k
- U15: value 74AHC541 -> 74AHCT541
Connections:
- net +5V: now also C51.1
- net GND: now also C51.2
- no-connect marks 0 -> 1
Changed lines of the file:
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@@
 	)
 	(junction
+		(at 38.1 25.4)
+		(diameter 0)
+		(color 0 0 0 0)
+	)
+	(junction
 		(at 186.69 40.64)
 		(diameter 0)
@@
 		(color 0 0 0 0)
 	)
+	(no_connect
+		(at 279.4 41.91)
+	)
 	(wire
 		(pts
@@
 	(wire
 		(pts
+			(xy 44.45 25.4) (xy 38.1 25.4)
+		)
+		(stroke
+			(width 0)
+			(type default)
+		)
+	)
+	(wire
+		(pts
 			(xy 57.15 134.62) (xy 57.15 135.89)
 		)
@@
 			)
 		)
-		(property "Value" "BZT52Bxx"
+		(property "Value" "BZT52C6V2"
 			(at 92.71 142.2399 90)
 			(effects
@@
 	)
 	(symbol
+		(lib_id "Device:C")
+		(at 48.26 25.4 90)
+		(unit 1)
+		(exclude_from_sim no)
+		(in_bom yes)
+		(on_board yes)
+		(dnp no)
+		(fields_autoplaced yes)
+		(property "Reference" "C51"
+			(at 48.26 17.78 90)
+			(effects
+				(font
+					(size 1.27 1.27)
+				)
+			)
+		)
+		(property "Value" "100n"
+			(at 48.26 20.32 90)
+			(effects
+				(font
+					(size 1.27 1.27)
+				)
+			)
+		)
+		(property "Footprint" "Capacitor_SMD:C_0603_1608Metric"
+			(at 52.07 24.4348 0)
+			(effects
+				(font
+					(size 1.27 1.27)
+				)
+				(hide yes)
+			)
+		)
+		(property "Datasheet" "~"
+			(at 48.26 25.4 0)
+			(effects
+				(font
+					(size 1.27 1.27)
+				)
+				(hide yes)
+			)
+		)
+		(property "Description" "Unpolarized capacitor"
+			(at 48.26 25.4 0)
+			(effects
+				(font
+					(size 1.27 1.27)
+				)
+				(hide yes)
+			)
+		)
+		(property "JLCPCB Part #" ""
+			(at 48.26 25.4 0)
+			(effects
+				(font
+					(size 1.27 1.27)
+				)
+				(hide yes)
+			)
+		)
+		(property "Sim.Device" ""
+			(at 48.26 25.4 0)
+			(effects
+				(font
+					(size 1.27 1.27)
+				)
+				(hide yes)
+			)
+		)
+		(property "LCSC Part Number" "C1525"
+			(at 48.26 25.4 0)
+			(effects
+				(font
+					(size 1.27 1.27)
+				)
+				(hide yes)
+			)
+		)
+		(property "LCSC" ""
+			(at 48.26 25.4 0)
+			(effects
+				(font
+					(size 1.27 1.27)
+				)
+				(hide yes)
+			)
+		)
+		(property "Manufacturer" ""
+			(at 48.26 25.4 0)
+			(effects
+				(font
+					(size 1.27 1.27)
+				)
+				(hide yes)
+			)
+		)
+		(property "Manufacturer Part" ""
+			(at 48.26 25.4 0)
+			(effects
+				(font
+					(size 1.27 1.27)
+				)
+				(hide yes)
+			)
+		)
+		(pin "2"
+		)
+		(pin "1"
+		)
+		(instances
+			(project "M.I.A."
+				(path "/4d55825e-4251-44bf-9376-9abd9228f348/e00a3c08-9b0c-4c55-ba07-ab188e60e59b"
+					(reference "C51")
+					(unit 1)
+				)
+			)
+		)
+	)
+	(symbol
 		(lib_id "Device:R")
 		(at 57.15 140.97 0)
@@
 			)
 		)
-		(property "Value" "1M"
+		(property "Value" "10k"
 			(at 59.69 142.2399 0)
 			(effects
@@
 			)
 		)
-		(property "Value" "BZT52Bxx"
+		(property "Value" "BZT52C6V2"
 			(at 92.71 176.5299 90)
 			(effects
@@
 			)
 		)
-		(property "Value" "5M"
+		(property "Value" "50k"
 			(at 118.11 132.0799 0)
 			(effects
@@
 			)
 		)
-		(property "Value" "5M"
+		(property "Value" "50k"
 			(at 118.11 166.3699 0)
 			(effects
@@
 			)
 		)
-		(property "Value" "BZT52Bxx"
+		(property "Value" "BZT52C6V2"
 			(at 34.29 176.5299 90)
 			(effects
@@
 			)
 		)
-		(property "Value" "1M"
+		(property "Value" "10k"
 			(at 59.69 176.5299 0)
 			(effects
@@
 			)
 		)
-		(property "Value" "BZT52Bxx"
+		(property "Value" "BZT52C6V2"
 			(at 34.29 142.2399 90)
 			(effects
@@
 		(on_board yes)
 		(dnp no)
-		(fields_autoplaced yes)
 		(property "Reference" "U15"
-			(at 40.2433 25.4 0)
+			(at 24.13 24.638 0)
 			(effects
 				(font
@@
 			)
 		)
-		(property "Value" "74AHC541"
-			(at 40.2433 27.94 0)
+		(property "Value" "74AHCT541"
+			(at 24.13 27.178 0)
 			(effects
 				(font
@@
 			)
 		)
-		(property "Value" "1M"
+		(property "Value" "10k"
 			(at 118.11 176.5299 0)
 			(effects
@@
 			)
 		)
-		(property "Value" "5M"
+		(property "Value" "50k"
 			(at 59.69 166.3699 0)
 			(effects
@@
 			)
 		)
-		(property "Value" "1M"
+		(property "Value" "10k"
 			(at 118.11 142.2399 0)
 			(effects
@@
 			)
 		)
-		(property "Value" "5M"
+		(property "Value" "50k"
 			(at 59.69 132.0799 0)
 			(effects
@@
 					(unit 1)
 				)
+			)
+		)
+	)
+	(symbol
+		(lib_id "power:GND")
+		(at 52.07 25.4 0)
+		(unit 1)
+		(exclude_from_sim no)
+		(in_bom yes)
+		(on_board yes)
+		(dnp no)
+		(property "Reference" "#PWR0191"
+			(at 52.07 31.75 0)
+			(effects
+				(font
+					(size 1.27 1.27)
+				)
+				(hide yes)
+			)
+		)
+		(property "Value" "GND"
+			(at 52.07 29.21 0)
+			(effects
+				(font
+					(size 1.27 1.27)
+				)
+			)
+		)
+		(property "Footprint" ""
+			(at 52.07 25.4 0)
+			(effects
+				(font
+					(size 1.27 1.27)
+				)
+				(hide yes)
+			)
+		)
+		(property "Datasheet" ""
+			(at 52.07 25.4 0)
+			(effects
+				(font
+					(size 1.27 1.27)
+				)
+				(hide yes)
+			)
+		)
+		(property "Description" "Power symbol creates a global label with name \"GND\" , ground"
+			(at 52.07 25.4 0)
+			(effects
+				(font
+					(size 1.27 1.27)
+				)
+				(hide yes)
+			)
+		)
+		(pin "1"
+		)
+		(instances
+			(project "M.I.A."
+				(path "/4d55825e-4251-44bf-9376-9abd9228f348/e00a3c08-9b0c-4c55-ba07-ab188e60e59b"
+					(reference "#PWR0191")
+					(unit 1)
+				)
